File: can.kicad_sch (KiCad schematic)
At the start: 16 parts, among them J601 Conn_01x01, J602 Conn_01x01, Q601 2N7002, Q602 AO3401A, Q603 AO3401A, U301 TJA1462ATK/0Z

Commit message: redesing board
Parts:
- renumbered C602 to C301, C601 to C302, C603 to C303, D3 to D301, J601 to J301, J602 to J302, Q601 to Q301, Q602 to Q302, Q603 to Q303, R603 to R301, R601 to R302, R602 to R303, R604 to R304, R605 to R305, R606 to R306
Changed lines of the file:
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@@
 		(dnp no)
 		(fields_autoplaced yes)
-		(property "Reference" "Q602"
+		(property "Reference" "Q302"
 			(at 151.765 100.33 0)
 			(effects
@@
 			(project "CAN2GPIO2"
 				(path "/48fe87cd-0661-436a-93bb-f175c4d0f54e/6c759029-600a-4c3d-8c40-75cdb4e7f614"
-					(reference "Q602")
+					(reference "Q302")
 					(unit 1)
 				)
@@
 		(dnp no)
 		(fields_autoplaced yes)
-		(property "Reference" "#PWR0602"
+		(property "Reference" "#PWR0301"
 			(at 52.07 96.52 0)
 			(effects
@@
 			(project "CAN2GPIO2"
 				(path "/48fe87cd-0661-436a-93bb-f175c4d0f54e/6c759029-600a-4c3d-8c40-75cdb4e7f614"
-					(reference "#PWR0602")
+					(reference "#PWR0301")
 					(unit 1)
 				)
@@
 		(dnp no)
 		(fields_autoplaced yes)
-		(property "Reference" "R603"
+		(property "Reference" "R301"
 			(at 139.7 49.911 90)
 			(effects
@@
 			(project "CAN2GPIO2"
 				(path "/48fe87cd-0661-436a-93bb-f175c4d0f54e/6c759029-600a-4c3d-8c40-75cdb4e7f614"
-					(reference "R603")
+					(reference "R301")
 					(unit 1)
 				)
@@
 		(dnp no)
 		(fields_autoplaced yes)
-		(property "Reference" "J601"
+		(property "Reference" "J301"
 			(at 220.345 81.28 0)
 			(effects
@@
 			(project "CAN2GPIO2"
 				(path "/48fe87cd-0661-436a-93bb-f175c4d0f54e/6c759029-600a-4c3d-8c40-75cdb4e7f614"
-					(reference "J601")
+					(reference "J301")
 					(unit 1)
 				)
@@
 		(on_board yes)
 		(dnp no)
-		(property "Reference" "C603"
+		(property "Reference" "C303"
 			(at 152.781 114.427 0)
 			(effects
@@
 			(project "CAN2GPIO2"
 				(path "/48fe87cd-0661-436a-93bb-f175c4d0f54e/6c759029-600a-4c3d-8c40-75cdb4e7f614"
-					(reference "C603")
+					(reference "C303")
 					(unit 1)
 				)
@@
 		(dnp no)
 		(fields_autoplaced yes)
-		(property "Reference" "#PWR0301"
+		(property "Reference" "#PWR0302"
 			(at 69.85 81.28 0)
 			(effects
@@
 			(project "rc_ble"
 				(path "/48fe87cd-0661-436a-93bb-f175c4d0f54e/6c759029-600a-4c3d-8c40-75cdb4e7f614"
-					(reference "#PWR0301")
+					(reference "#PWR0302")
 					(unit 1)
 				)
@@
 		(dnp no)
 		(fields_autoplaced yes)
-		(property "Reference" "R604"
+		(property "Reference" "R304"
 			(at 156.845 90.17 0)
 			(effects
@@
 			(project "CAN2GPIO2"
 				(path "/48fe87cd-0661-436a-93bb-f175c4d0f54e/6c759029-600a-4c3d-8c40-75cdb4e7f614"
-					(reference "R604")
+					(reference "R304")
 					(unit 1)
 				)
@@
 		(dnp no)
 		(fields_autoplaced yes)
-		(property "Reference" "#PWR0605"
+		(property "Reference" "#PWR0306"
 			(at 160.02 127 0)
 			(effects
@@
 			(project "CAN2GPIO2"
 				(path "/48fe87cd-0661-436a-93bb-f175c4d0f54e/6c759029-600a-4c3d-8c40-75cdb4e7f614"
-					(reference "#PWR0605")
+					(reference "#PWR0306")
 					(unit 1)
 				)
@@
 		(dnp no)
 		(fields_autoplaced yes)
-		(property "Reference" "C601"
+		(property "Reference" "C302"
 			(at 114.3 102.8763 0)
 			(effects
@@
 			(project "CAN2GPIO2"
 				(path "/48fe87cd-0661-436a-93bb-f175c4d0f54e/6c759029-600a-4c3d-8c40-75cdb4e7f614"
-					(reference "C601")
+					(reference "C302")
 					(unit 1)
 				)
@@
 		(dnp no)
 		(fields_autoplaced yes)
-		(property "Reference" "#PWR0302"
+		(property "Reference" "#PWR0304"
 			(at 144.78 78.74 0)
 			(effects
@@
 			(project "rc_ble"
 				(path "/48fe87cd-0661-436a-93bb-f175c4d0f54e/6c759029-600a-4c3d-8c40-75cdb4e7f614"
-					(reference "#PWR0302")
+					(reference "#PWR0304")
 					(unit 1)
 				)
@@
 		(dnp no)
 		(fields_autoplaced yes)
-		(property "Reference" "#PWR0604"
+		(property "Reference" "#PWR0305"
 			(at 152.4 81.28 0)
 			(effects
@@
 			(project "CAN2GPIO2"
 				(path "/48fe87cd-0661-436a-93bb-f175c4d0f54e/6c759029-600a-4c3d-8c40-75cdb4e7f614"
-					(reference "#PWR0604")
+					(reference "#PWR0305")
 					(unit 1)
 				)
@@
 		(dnp no)
 		(fields_autoplaced yes)
-		(property "Reference" "R601"
+		(property "Reference" "R302"
 			(at 139.7 60.96 90)
 			(effects
@@
 			(project "CAN2GPIO2"
 				(path "/48fe87cd-0661-436a-93bb-f175c4d0f54e/6c759029-600a-4c3d-8c40-75cdb4e7f614"
-					(reference "R601")
+					(reference "R302")
 					(unit 1)
 				)
@@
 		(dnp no)
 		(fields_autoplaced yes)
-		(property "Reference" "Q603"
+		(property "Reference" "Q303"
 			(at 177.8 100.33 0)
 			(effects
@@
 			(project "CAN2GPIO2"
 				(path "/48fe87cd-0661-436a-93bb-f175c4d0f54e/6c759029-600a-4c3d-8c40-75cdb4e7f614"
-					(reference "Q603")
+					(reference "Q303")
 					(unit 1)
 				)
@@
 		(dnp no)
 		(fields_autoplaced yes)
-		(property "Reference" "J602"
+		(property "Reference" "J302"
 			(at 219.71 85.09 0)
 			(effects
@@
 			(project "CAN2GPIO2"
 				(path "/48fe87cd-0661-436a-93bb-f175c4d0f54e/6c759029-600a-4c3d-8c40-75cdb4e7f614"
-					(reference "J602")
+					(reference "J302")
 					(unit 1)
 				)
@@
 		(dnp no)
 		(fields_autoplaced yes)
-		(property "Reference" "#PWR017"
+		(property "Reference" "#PWR0308"
 			(at 196.85 106.68 0)
 			(effects
@@
 			(project "can2gpio"
 				(path "/48fe87cd-0661-436a-93bb-f175c4d0f54e/6c759029-600a-4c3d-8c40-75cdb4e7f614"
-					(reference "#PWR017")
+					(reference "#PWR0308")
 					(unit 1)
 				)
@@
 		(dnp no)
 		(fields_autoplaced yes)
-		(property "Reference" "#PWR0601"
+		(property "Reference" "#PWR0303"
 			(at 111.76 114.3 0)
 			(effects
@@
 			(project "CAN2GPIO2"
 				(path "/48fe87cd-0661-436a-93bb-f175c4d0f54e/6c759029-600a-4c3d-8c40-75cdb4e7f614"
-					(reference "#PWR0601")
+					(reference "#PWR0303")
 					(unit 1)
 				)
@@
 		(dnp no)
 		(fields_autoplaced yes)
-		(property "Reference" "R605"
+		(property "Reference" "R305"
 			(at 172.085 114.3 0)
 			(effects
@@
 			(project "CAN2GPIO2"
 				(path "/48fe87cd-0661-436a-93bb-f175c4d0f54e/6c759029-600a-4c3d-8c40-75cdb4e7f614"
-					(reference "R605")
+					(reference "R305")
 					(unit 1)
 				)
@@
 		(dnp no)
 		(fields_autoplaced yes)
-		(property "Reference" "C602"
+		(property "Reference" "C301"
 			(at 54.61 85.0963 0)
 			(effects
@@
 			(project "CAN2GPIO2"
 				(path "/48fe87cd-0661-436a-93bb-f175c4d0f54e/6c759029-600a-4c3d-8c40-75cdb4e7f614"
-					(reference "C602")
+					(reference "C301")
 					(unit 1)
 				)
@@
 		(dnp no)
 		(fields_autoplaced yes)
-		(property "Reference" "#PWR0606"
+		(property "Reference" "#PWR0307"
 			(at 170.18 127 0)
 			(effects
@@
 			(project "CAN2GPIO2"
 				(path "/48fe87cd-0661-436a-93bb-f175c4d0f54e/6c759029-600a-4c3d-8c40-75cdb4e7f614"
-					(reference "#PWR0606")
+					(reference "#PWR0307")
 					(unit 1)
 				)
@@
 		(on_board yes)
 		(dnp no)
-		(property "Reference" "R602"
+		(property "Reference" "R303"
 			(at 145.415 69.85 0)
 			(effects
@@
 			(project "CAN2GPIO2"
 				(path "/48fe87cd-0661-436a-93bb-f175c4d0f54e/6c759029-600a-4c3d-8c40-75cdb4e7f614"
-					(reference "R602")
+					(reference "R303")
 					(unit 1)
 				)
@@
 		(on_board yes)
 		(dnp no)
-		(property "Reference" "D3"
+		(property "Reference" "D301"
 			(at 202.438 96.774 0)
 			(effects
@@
 			(project "can2gpio"
 				(path "/48fe87cd-0661-436a-93bb-f175c4d0f54e/6c759029-600a-4c3d-8c40-75cdb4e7f614"
-					(reference "D3")
+					(reference "D301")
 					(unit 1)
 				)
@@
 		(dnp no)
 		(fields_autoplaced yes)
-		(property "Reference" "R606"
+		(property "Reference" "R306"
 			(at 175.895 90.17 0)
 			(effects
@@
 			(project "CAN2GPIO2"
 				(path "/48fe87cd-0661-436a-93bb-f175c4d0f54e/6c759029-600a-4c3d-8c40-75cdb4e7f614"
-					(reference "R606")
+					(reference "R306")
 					(unit 1)
 				)
@@
 		(dnp no)
 		(fields_autoplaced yes)
-		(property "Reference" "Q601"
+		(property "Reference" "Q301"
 			(at 158.75 66.04 90)
 			(effects
@@
 			(project "CAN2GPIO2"
 				(path "/48fe87cd-0661-436a-93bb-f175c4d0f54e/6c759029-600a-4c3d-8c40-75cdb4e7f614"
-					(reference "Q601")
-					(unit 1)
-				)
+					(reference "Q301")
+					(unit 1)
+				)

Commit message: PCBA ready
Parts:
- C303: value 4.7pF -> 10pF
Changed lines of the file:
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@@
 			)
 		)
-		(property "Value" "4.7pF"
+		(property "Value" "10pF"
 			(at 152.781 116.713 0)
 			(effects
