File: rc_ble.kicad_pcb (KiCad board)
At the start: 2 copper layers, 44 parts, among them J3 SWD, J601 Conn_01x01, J602 Conn_01x01, Q601 2N7002, Q602 AO3401A, Q603 AO3401A, U102 TLV75533PDBV, U103 TXB0102DCU, U17 NEO-8M, U2 MCP2518FD-xQBB, U301 TJA1462ATK/0Z, Y1 20Mhz

Commit message: wip
Parts:
- removed C7, C8: 0.1uF, Capacitor_SMD:C_0603_1608Metric
- added C104: C_Polarized_Small, Capacitor_THT:CP_Radial_D5.0mm_P2.50mm, F.Cu at (110.5, 81.1)
- added D101: D_Schottky_Small, Diode_SMD:D_SOD-323_HandSoldering, F.Cu at (111.4, 87.9)
- added J101: Conn_Coaxial_Power, Connector_Coaxial:SMA_Amphenol_132134_Vertical, F.Cu at (98.9, 91.5)
- added L2: 27nH, Inductor_SMD:L_0805_2012Metric_Pad1.15x1.40mm_HandSolder, F.Cu at (105.1, 91.5)
- added R106: 33, Resistor_SMD:R_0603_1608Metric, F.Cu at (136.5, 66.7)
- added R107: 33, Resistor_SMD:R_0603_1608Metric, F.Cu at (133.9, 66.7)
- added R108: 33, Resistor_SMD:R_0603_1608Metric, F.Cu at (129.7, 67.7)
- added R109: 10K, Resistor_SMD:R_0603_1608Metric, F.Cu at (124.6, 70.1)
- U17: footprint ublox:NEO-M8N -> RF_GPS:ublox_NEO
- moved C105 52.6 mm to (132.7, 97.8)
- moved C106 45.1 mm to (131.7, 91.5)
- moved C2 37.8 mm to (128.5, 75.0), turned to -90 degrees
- moved J601 31.1 mm to (96.9, 72.2)
- moved C1 30.0 mm to (126.7, 75.2), turned to -90 degrees
- moved R104 29.9 mm to (111.3, 84.2), turned to -90 degrees
- moved C4 28.0 mm to (122.3, 69.2), turned to 180 degrees
- moved J602 26.4 mm to (96.9, 67.4)
- moved C5 24.7 mm to (117.2, 73.2), turned to 90 degrees
- moved D3 23.8 mm to (99.7, 69.8), turned to 180 degrees
- moved C3 23.6 mm to (122.1, 67.5), turned to 180 degrees
- moved R601 22.3 mm to (124.2, 78.7), turned to -90 degrees
- moved C603 21.9 mm to (103.1, 77.1), turned to 180 degrees
- moved Q601 21.2 mm to (119.9, 78.7), turned to 180 degrees
- moved R602 19.3 mm to (122.6, 78.7), turned to -90 degrees
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Connections:
- U1 pad 1: GND_ISO -> GND
- U1 pad 10: unconnected-(U1-P1.02-Pad10) -> Net-(U1-P1.02)
- U1 pad 11: GND_ISO -> GND
- U1 pad 12: GND_ISO -> GND
- U1 pad 22: unconnected-(U1-P0.20-Pad22) -> /MCP_RST
- U1 pad 24: unconnected-(U1-P1.07-Pad24) -> /GPS_ENABLE
- U1 pad 3: unconnected-(U1-P1.03-Pad3) -> /MCP_INT
- U1 pad 30: unconnected-(U1-P1.06-Pad30) -> /GPS_RX
- U1 pad 31: unconnected-(U1-P0.27-Pad31) -> /GPS_TX
- U1 pad 32: unconnected-(U1-RST-Pad32) -> /RST
- U1 pad 55: unconnected-(U1-P1.04-Pad55) -> /MCP_SPI_CS
- U1 pad 8: unconnected-(U1-P1.00-Pad8) -> Net-(U1-P1.00)
- U1 pad 9: unconnected-(U1-P1.01-Pad9) -> Net-(U1-P1.01)
- U103 pad 1: /GPS_TX -> /GPS_RX
- U103 pad 4: /ublox/GPS_TX -> /ublox/GPS_RX
- U103 pad 5: /ublox/GPS_RX -> /ublox/GPS_TX
- U103 pad 8: /GPS_RX -> /GPS_TX
Routing:
- net GND: track 0.00 -> 39.7 mm, vias 0 -> 19
- net /GPS_TX: track 0.00 -> 19.9 mm
- net /GPS_RX: track 0.00 -> 19.4 mm
- net /ublox/GPS_RF: track 0.00 -> 19.2 mm
- net /GPS_POWER: track 0.00 -> 19.1 mm
- net /MCP_SPI_MISO: track 0.00 -> 18.7 mm
- net Net-(U2-~{INT1}/GPIO1): track 0.00 -> 17.3 mm
- net /MCP_SPI_MOSI: track 0.00 -> 15.2 mm
- net /CAN/CAN1_HI: track 0.00 -> 14.5 mm
- net /CAN/CAN1_LOW: track 0.00 -> 14.1 mm
- net /ublox/GPS_RX: track 0.00 -> 12.8 mm
- net /ublox/GPS_TX: track 0.00 -> 12.3 mm
- net /MCP_RST: track 0.00 -> 12.0 mm
- net /3V3: track 0.00 -> 11.9 mm
- net /SWD_CLK: track 0.00 -> 11.6 mm
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- added copper zone on B.Cu, net GND
- added copper zone on F.Cu, net GND
Other:
- board outline added: 55.9 x 36.1 mm

Commit message: redesing board
Parts:
- added C110: 10nF, Capacitor_SMD:C_0603_1608Metric, F.Cu at (100.0, 91.4)
- added C111: 10uF, Capacitor_SMD:C_0603_1608Metric, F.Cu at (116.4, 98.1)
- added C112: 10nF, Capacitor_SMD:C_0603_1608Metric, F.Cu at (123.0, 98.9)
- added C114: 2.2uF, Capacitor_SMD:C_0603_1608Metric, F.Cu at (123.7, 97.3)
- added C401: 10uF, Capacitor_SMD:C_0805_2012Metric, F.Cu at (107.8, 91.7)
- added C402: 0.1uF, Capacitor_SMD:C_0805_2012Metric, F.Cu at (115.8, 94.1)
- added C403: 10uF, Capacitor_SMD:C_0805_2012Metric, F.Cu at (108.4, 98.1)
- added C404: 10uF, Capacitor_SMD:C_0805_2012Metric, F.Cu at (106.2, 98.1)
- added D102: WS2812B-2020, LED_SMD:LED_WS2812B-2020_PLCC4_2.0x2.0mm, F.Cu at (135.5, 65.0)
- added D103: WS2812B-2020, LED_SMD:LED_WS2812B-2020_PLCC4_2.0x2.0mm, F.Cu at (128.7, 65.0)
- added D104: BZT52C16S, Diode_SMD:D_SOD-323_HandSoldering, F.Cu at (101.8, 88.5)
- added D401: SS14FL, Diode_SMD:D_SMA, F.Cu at (106.0, 94.5)
- added H101: MountingHole_Pad, MountingHole:MountingHole_2.2mm_M2_Pad_Via, F.Cu at (144.0, 65.7)
- added H102: MountingHole_Pad, MountingHole:MountingHole_2.2mm_M2_Pad_Via, F.Cu at (97.6, 98.3)
- added J102: Vin, Connector_PinHeader_2.54mm:PinHeader_1x01_P2.54mm_Vertical, F.Cu at (97.2, 83.8)
- added J103: Gnd, Connector_PinHeader_2.54mm:PinHeader_1x01_P2.54mm_Vertical, F.Cu at (97.2, 80.2)
- added L401: 22uH, inductor:FNR5040S220MT, F.Cu at (112.1, 96.9)
- added Q101: AO3401A, Package_TO_SOT_SMD:SOT-23, F.Cu at (100.8, 84.5)
- added R107: 10K, Resistor_SMD:R_0603_1608Metric, F.Cu at (100.0, 88.0)
- added R401: 100K, Resistor_SMD:R_0603_1608Metric, F.Cu at (109.8, 89.8)
- added R402: 54.9K, Resistor_SMD:R_0603_1608Metric, F.Cu at (115.2, 90.1)
- added R403: 10K, Resistor_SMD:R_0603_1608Metric, F.Cu at (112.8, 89.8)
- added TP101: 5V, TestPoint:TestPoint_Pad_1.0x1.0mm, F.Cu at (102.6, 99.1)
- added TP102: 3V3, TestPoint:TestPoint_Pad_1.0x1.0mm, F.Cu at (124.1, 74.5)
- added U105: LP2985-3.3, Package_TO_SOT_SMD:SOT-23-5, F.Cu at (119.4, 98.2)
- added U401: LMR16006Y, Package_TO_SOT_SMD:SOT-23-6, F.Cu at (112.2, 92.3)
- C104: footprint Capacitor_THT:CP_Radial_D5.0mm_P2.50mm -> Capacitor_THT:CP_Radial_D8.0mm_P3.50mm
- L201: renamed from L2; footprint Inductor_SMD:L_0805_2012Metric_Pad1.15x1.40mm_HandSolder -> Inductor_SMD:L_0805_2012Metric
- R201: renamed from R40; footprint Resistor_SMD:R_1206_3216Metric -> Resistor_SMD:R_0603_1608Metric
- moved JP101 38.7 mm to (135.9, 97.3), turned to 0 degrees
- moved R103 33.8 mm to (136.7, 95.2), turned to 180 degrees
- moved R104 33.1 mm to (133.1, 95.2)
- moved Q303 30.7 mm to (122.5, 89.9), turned to -90 degrees
- moved C201 27.5 mm to (97.7, 67.8)
- moved R201 27.0 mm to (101.9, 66.7), turned to 0 degrees
- moved C106 26.8 mm to (124.2, 65.8)
- moved C108 26.8 mm to (125.1, 72.0)
- moved U102 26.8 mm to (124.1, 68.9)
- moved R306 25.4 mm to (117.3, 84.7), turned to 0 degrees
- moved L201 24.4 mm to (99.5, 67.8), turned to 90 degrees
- moved C301 24.1 mm to (131.4, 86.7)
- moved U301 24.1 mm to (127.6, 87.0)
- moved C302 24.0 mm to (124.6, 84.8)
- moved C103 23.9 mm to (131.1, 92.5)
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- renumbered C6 to C101, C3 to C102, C5 to C103, C4 to C105, C102 to C107, C105 to C108, C101 to C109, C1 to C113, C2 to C115, C40 to C201, C49 to C202, C602 to C301, C601 to C302, C603 to C303, D3 to D301, J3 to J104, J601 to J301, J602 to J302, JP102 to JP101, Q601 to Q301, Q602 to Q302, Q603 to Q303, R109 to R101, R104 to R102, R105 to R103, R101 to R104, R102 to R105, R103 to R106, R106 to R108, R108 to R109, R107 to R110, R603 to R301, R601 to R302, R602 to R303, R604 to R304, R605 to R305, R606 to R306, U2 to U101, U103 to U102, U102 to U103, U1 to U104, U17 to U201, Y1 to Y101
Connections:
- J104 pad 2: unconnected-(J3-Pin_2-Pad2) -> /RST
- J104 pad 6: unconnected-(J3-Pin_6-Pad6) -> GND
- J104 pad 9: unconnected-(J3-Pin_9-Pad9) -> GND
- R108 pad 1: Net-(U1-P1.00) -> Net-(U104-P0.21)
- R109 pad 1: Net-(U1-P1.02) -> Net-(U104-P0.27)
- R110 pad 1: Net-(U1-P1.01) -> Net-(U104-P1.06)
- U104 pad 10: Net-(U1-P1.02) -> /GPS_TX
- U104 pad 19: unconnected-(U1-P0.15_(QSPI)-Pad19) -> /GPS_ENABLE
- U104 pad 22: /MCP_RST -> /CAN_TERM
- U104 pad 24: /GPS_ENABLE -> /MCP_INT
- U104 pad 25: unconnected-(U1-P1.09-Pad25) -> /MCP_RST
- U104 pad 28: unconnected-(U1-P0.19-Pad28) -> /MCP_SPI_CS
- U104 pad 29: unconnected-(U1-P0.21-Pad29) -> Net-(U104-P0.21)
- U104 pad 3: /MCP_INT -> unconnected-(U104-P1.03-Pad3)
- U104 pad 30: /GPS_RX -> Net-(U104-P1.06)
- U104 pad 31: /GPS_TX -> Net-(U104-P0.27)
- U104 pad 55: /MCP_SPI_CS -> unconnected-(U104-P1.04-Pad55)
- U104 pad 8: Net-(U1-P1.00) -> /LED_CONTROL
- U104 pad 9: Net-(U1-P1.01) -> /GPS_RX
Routing:
- net Net-(U101-~{INT1}/GPIO1): track 17.3 -> 0.00 mm
- net /ublox/GPS_VBAT: track 0.00 -> 13.2 mm
- net /12V: track 0.00 -> 13.1 mm
- net /RST: track 0.00 -> 12.8 mm, vias 0 -> 2
- net /MCP_SPI_MISO: track 18.7 -> 6.05 mm
- net /ublox/GPS_TX: track 12.3 -> 0.00 mm
- net GND: track 39.7 -> 27.8 mm, vias 19 -> 21
- net /MCP_INT: track 0.00 -> 11.0 mm, vias 0 -> 2
- net Net-(Q301-D): track 2.22 -> 11.7 mm
- net /GPS_POWER: track 19.1 -> 27.9 mm
- net Net-(Q303-D): track 2.45 -> 10.3 mm, vias 0 -> 2
- net /MCP_SPI_CS: track 1.68 -> 9.22 mm
- net /MCP_SPI_MOSI: track 15.2 -> 7.95 mm
- net /GPS_TX: track 19.9 -> 13.4 mm
- net /CAN_TERM: track 0.00 -> 5.59 mm
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- added copper zone on F.Cu, net /5V
- added copper zone on In2.Cu, net /5V
- added copper zone on In1.Cu, net GND
Other:
- board size 55.9 x 36.1 mm -> 52.5 x 38.6 mm
- copper layers 2 -> 4

Commit message: wip
Parts:
- moved JP101 4.42 mm to (131.9, 99.2)
- moved R107 2.03 mm to (99.8, 90.0)
- moved R103 1.96 mm to (134.7, 95.5)
- moved C110 1.92 mm to (101.3, 90.1), turned to -90 degrees
- moved R104 1.55 mm to (131.9, 96.3), turned to -90 degrees
- moved D104 1.27 mm to (101.0, 87.5), turned to 180 degrees
- moved R302 0.62 mm to (127.1, 84.3)
Connections:
- U102 pad 1: /GPS_RX -> /GPS_TX
- U102 pad 4: /ublox/GPS_RX -> /ublox/GPS_TX
- U102 pad 5: /ublox/GPS_TX -> /ublox/GPS_RX
- U102 pad 8: /GPS_TX -> /GPS_RX
- U104 pad 10: /GPS_TX -> /GPS_RX
- U104 pad 9: /GPS_RX -> /GPS_TX
Routing:
- net /5V: track 5.48 -> 149.3 mm, vias 5 -> 21
- net GND: track 27.8 -> 61.5 mm, vias 21 -> 77
- net /CAN/CAN1_LOW: track 12.4 -> 36.5 mm, vias 0 -> 1
- net /CAN/CAN1_HI: track 12.5 -> 34.9 mm, vias 0 -> 1
- net /CAN/CAN1S: track 0.00 -> 14.6 mm, vias 0 -> 2
- net /ublox/GPS_TX: track 0.00 -> 14.5 mm
- net Net-(Q301-G): track 1.82 -> 16.1 mm, vias 0 -> 2
- net /3V3: track 17.3 -> 24.7 mm, vias 0 -> 19
- net /ublox/GPS_RX: track 16.2 -> 12.0 mm
- net Net-(U101-~{INT1}/GPIO1): track 0.00 -> 4.15 mm
- net Net-(U401-FB): track 0.00 -> 3.38 mm
- net Net-(U401-CB): track 0.00 -> 2.38 mm
- net Net-(JP101-C): track 0.00 -> 2.04 mm
- net Net-(Q302-S): track 0.00 -> 1.91 mm
- net /GPS_TX: track 13.4 -> 15.2 mm
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- added copper zone on F.Cu, net /3V3
- added copper zone on In2.Cu, net /3V3
- added copper zone on In1.Cu, net /5V
- added copper zone on In2.Cu, net GND
- added copper zone on F.Cu, net Net-(D401-K)

Commit message: wip
Parts:
- added LOGO101: ~, logo:logo_github, B.Cu at (138.1, 83.2)
- added LOGO102: ~, logo:logo_15x9, B.Cu at (138.6, 96.9)
Routing:
- net /5V: track 149.3 -> 146.0 mm
Other:
- outline, holes or cut-outs redrawn
- board text added: "+"
- board text added: "-"
- board text added: "12V"
- board text added: "3V3"
- board text added: "5V"
- board text added: "CANH"
- board text added: "CANL"
- board text added: "GND"
- board text added: "PD"
- board text added: "PU"

Commit message: VDDH pin
Connections:
- U104 pad 14: unconnected-(U104-VDDH-Pad14) -> /3V3
Routing:
- net /3V3: track 24.7 -> 29.6 mm

Commit message: PCBA ready
Parts:
- C101, C103: value 12pF -> 8pF
- C201: value 0.01uF -> 10nF
- C303: value 4.7pF -> 10pF
Changed lines of the file:
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@@
 			)
 		)
+		(property "LCSC" "C22775"
+			(at 0 0 0)
+			(layer "F.SilkS")
+			(hide yes)
+			(effects
+				(font
+					(size 1.27 1.27)
+					(thickness 0.15)
+				)
+			)
+		)
 		(property ki_fp_filters "R_*")
 		(sheetname "/")
@@
 			)
 		)
+		(property "LCSC" "C42372555"
+			(at 0 0 0)
+			(layer "F.SilkS")
+			(hide yes)
+			(effects
+				(font
+					(size 1.27 1.27)
+					(thickness 0.15)
+				)
+			)
+		)
 		(property ki_fp_filters "Connector*:*_2x??_*")
 		(sheetname "/")
@@
 			)
 		)
+		(property "LCSC" "C440198"
+			(at 0 0 0)
+			(layer "F.SilkS")
+			(hide yes)
+			(effects
+				(font
+					(size 1.27 1.27)
+					(thickness 0.15)
+				)
+			)
+		)
 		(property ki_fp_filters "C_*")
 		(sheetname "/")
@@
 		(sheetname "/CAN/")
 		(sheetfile "can.kicad_sch")
-		(attr through_hole exclude_from_bom)
+		(attr through_hole exclude_from_pos_files exclude_from_bom)
 		(fp_line
 			(start -1.38 -1.38)
@@
 			)
 		)
-		(property "Value" "12pF"
+		(property "Value" "8pF"
 			(at 0 1.43 90)
 			(layer "F.Fab")
@@
 			)
 		)
+		(property "LCSC" "C28233"
+			(at 0 0 0)
+			(layer "F.SilkS")
+			(hide yes)
+			(effects
+				(font
+					(size 1.27 1.27)
+					(thickness 0.15)
+				)
+			)
+		)
 		(property ki_fp_filters "C_*")
 		(sheetname "/ublox/")
@@
 			)
 		)
+		(property "LCSC" "C440198"
+			(at 0 0 0)
+			(layer "F.SilkS")
+			(hide yes)
+			(effects
+				(font
+					(size 1.27 1.27)
+					(thickness 0.15)
+				)
+			)
+		)
 		(property ki_fp_filters "C_*")
 		(sheetname "/")
@@
 			)
 		)
-		(property "Value" "12pF"
+		(property "Value" "8pF"
 			(at 0 1.43 90)
 			(layer "F.Fab")
@@
 			)
 		)
-		(property "Value" "0.01uF"
+		(property "Value" "10nF"
 			(at 0 1.43 90)
 			(layer "F.Fab")
@@
 			)
 		)
+		(property "LCSC" "C57112"
+			(at 0 0 0)
+			(layer "F.SilkS")
+			(hide yes)
+			(effects
+				(font
+					(size 1.27 1.27)
+					(thickness 0.15)
+				)
+			)
+		)
 		(property ki_fp_filters "C_*")
 		(sheetname "/ublox/")
@@
 		(sheetname "/")
 		(sheetfile "rc_ble.kicad_sch")
-		(attr through_hole exclude_from_bom)
+		(attr through_hole exclude_from_pos_files exclude_from_bom)
 		(fp_line
 			(start -1.38 -1.38)
@@
 		(sheetname "/")
 		(sheetfile "rc_ble.kicad_sch")
-		(attr through_hole exclude_from_bom)
+		(attr through_hole exclude_from_pos_files exclude_from_bom)
 		(fp_line
 			(start -1.38 -1.38)
@@
 		(sheetname "/")
 		(sheetfile "rc_ble.kicad_sch")
-		(attr smd)
+		(attr smd exclude_from_pos_files exclude_from_bom)
 		(fp_rect
 			(start -0.68 -15.68)
@@
 			)
 		)
+		(property "LCSC" "C14663"
+			(at 0 0 0)
+			(layer "F.SilkS")
+			(hide yes)
+			(effects
+				(font
+					(size 1.27 1.27)
+					(thickness 0.15)
+				)
+			)
+		)
 		(property ki_fp_filters "C_*")
 		(sheetname "/")
@@
 			)
 		)
+		(property "LCSC" "C440198"
+			(at 0 0 0)
+			(layer "F.SilkS")
+			(hide yes)
+			(effects
+				(font
+					(size 1.27 1.27)
+					(thickness 0.15)
+				)
+			)
+		)
 		(property ki_fp_filters "C_*")
 		(sheetname "/")
@@
 		(sheetname "/CAN/")
 		(sheetfile "can.kicad_sch")
-		(attr through_hole exclude_from_bom)
+		(attr through_hole exclude_from_pos_files exclude_from_bom)
 		(fp_line
 			(start -1.38 -1.38)
@@
 		(sheetname "/")
 		(sheetfile "rc_ble.kicad_sch")
-		(attr through_hole)
+		(attr through_hole exclude_from_pos_files exclude_from_bom)
 		(fp_line
 			(start -3.68 -1.8)
@@
 		(sheetname "/")
 		(sheetfile "rc_ble.kicad_sch")
-		(attr through_hole)
+		(attr through_hole exclude_from_pos_files exclude_from_bom)
 		(fp_line
 			(start 2.47 1.04)
@@
 			)
 		)
+		(property "LCSC" "C440198"
+			(at 0 0 0)
+			(layer "F.SilkS")
+			(hide yes)
+			(effects
+				(font
+					(size 1.27 1.27)
+					(thickness 0.15)
+				)
+			)
+		)
 		(property ki_fp_filters "C_*")
 		(sheetname "/")
@@
 			)
 		)
-		(property "Value" "4.7pF"
+		(property "Value" "10pF"
 			(at 0 1.43 90)
 			(layer "F.Fab")
@@
 			)
 		)
+		(property "LCSC" "C14663"
+			(at 0 0 0)
+			(layer "F.SilkS")
+			(hide yes)
+			(effects
+				(font
+					(size 1.27 1.27)
+					(thickness 0.15)
+				)
+			)
+		)
 		(property ki_fp_filters "C_*")
 		(sheetname "/")
@@
 		(sheetname "/")
 		(sheetfile "rc_ble.kicad_sch")
-		(attr board_only exclude_from_pos_files)
+		(attr board_only exclude_from_pos_files exclude_from_bom)
 		(fp_poly
 			(pts
