File: rc_ble.kicad_sch (KiCad schematic)
At the start: 0 parts

Commit message: wip
Parts:
- added C1, C101, C102, C3: 10uF, Capacitor_SMD:C_0805_2012Metric, symbol Device:C_Small
- added C104: C_Polarized_Small, symbol Device:C_Polarized_Small
- added C105, C106, C2, C4, C7, C8: 0.1uF, Capacitor_SMD:C_0603_1608Metric, symbol Device:C_Small
- added C5, C6: 12pF, Capacitor_SMD:C_0603_1608Metric, symbol Device:C_Small
- added D101: D_Schottky_Small, symbol Device:D_Schottky_Small
- added J101: Conn_Coaxial_Power, symbol Connector:Conn_Coaxial_Power
- added J3: SWD, Connector_PinHeader_1.27mm:PinHeader_2x05_P1.27mm_Vertical_SMD, symbol Connector_Generic:Conn_02x05_Odd_Even
- added JP102: CAN_ENABLE, Jumper:SolderJumper-3_P1.3mm_Open_RoundedPad1.0x1.5mm, symbol Jumper:SolderJumper_3_Open
- added R101, R102: 10K, Resistor_SMD:R_0603_1608Metric, symbol Device:R_Small
- added R103, R104, R105: 100, Resistor_SMD:R_0603_1608Metric, symbol Device:R_Small
- added U1: ~, holyiot_21069_nrf5340:nrf5340, symbol holyiot_21069:holyiot_21069_nfr5340
- added U102: TLV75533PDBV, Package_TO_SOT_SMD:SOT-23-5, symbol Regulator_Linear:TLV75533PDBV
- added U103: TXB0102DCU, Package_SO:VSSOP-8_2.3x2mm_P0.5mm, symbol Logic_LevelTranslator:TXB0102DCU
- added U2: MCP2518FD-xQBB, Package_DFN_QFN:DFN-14-1EP_3x4.5mm_P0.65mm_EP1.65x4.25mm, symbol Interface_CAN_LIN:MCP2518FD-xQBB
- added Y1: 20Mhz, Crystal:Crystal_SMD_3225-4Pin_3.2x2.5mm, symbol Device:Crystal_GND24_Small
Connections:
- new net: C5.1, U2.6 (OSC1), Y1.1
- new net: R105.1, U2.8 (~{INT1}/GPIO1)
- new net: R102.1, R103.1, U102.3 (EN)
- new net: C6.1, U2.5 (OSC2), Y1.3
- new net: JP102.2 (C), R101.2
- new net: D101.1 (K), R104.2
- new net 3V3: C1.1, C105.1, C2.1, C3.1, C4.1, C7.1, J3.3 (Pin_3), JP102.1 (A), U1.16 (VDD), U103.7 (VCCB), U2.14 (VDD)
- new net 5V: C101.1, C8.1, J3.1 (Pin_1), U102.1 (IN)
- new net CAN/CAN1RX: U2.2 (RXCAN)
- new net CAN/CAN1S: R101.1, R105.2
- new net CAN/CAN1TX: U2.1 (TXCAN)
- new net GND: C1.2, C101.2, C102.2, C104.2, C105.2, C106.2, C2.2, C3.2, C4.2, C5.2, C6.2, C7.2, C8.2, J101.2 (Ext), JP102.3 (B), R102.2, U102.2 (GND), U103.2 (GND), U2.15 (VSS), U2.7 (VSS), Y1.2, Y1.4
- new net GND_ISO: U1.1 (GND), U1.11 (GND), U1.12 (GND)
- new net GPS_ENABLE: R103.2
- new net GPS_POWER: C102.1, C106.1, D101.2 (A), U102.5 (OUT), U103.3 (VCCA), U103.6 (OE)
- new net GPS_RX: U103.8 (B1)
- new net GPS_TX: U103.1 (B2)
- new net MCP_INT: U2.4 (~{INT})
- new net MCP_RST: U2.9 (~{INT0}/GPIO0/XSTBY)
- new net MCP_SPI_CS: U2.13 (~{CS})
- new net MCP_SPI_MISO: U2.12 (SDO)
- new net MCP_SPI_MOSI: U2.11 (SDI)
- new net MCP_SPI_SCK: U2.10 (SCK)
- new net SWD_CLK: J3.7 (Pin_7), U1.36 (SWDCK)
- new net SWD_IO: J3.5 (Pin_5), U1.35 (SWDIO)
- new net ublox/GPS_RF: J101.1 (In)
- new net ublox/GPS_RX: U103.5 (A1)
- new net ublox/GPS_TX: U103.4 (A2)
- new net ublox/GPS_VBAT: C104.1, R104.1
- no-connect marks 0 -> 5
Other:
- added sheet CAN (can.kicad_sch)
- added sheet ublox (ubloxM8N.kicad_sch)
- note added: "CAN"
- note added: "GPS"

Commit message: wip
Parts:
- removed C7, C8: 0.1uF, Capacitor_SMD:C_0603_1608Metric, symbol Device:C_Small
- added R106, R107, R108: 33, Resistor_SMD:R_0603_1608Metric, symbol Device:R_Small
- added R109: 10K, Resistor_SMD:R_0603_1608Metric, symbol Device:R_Small
- C104: footprint (none) -> Capacitor_THT:CP_Radial_D5.0mm_P2.50mm
- D101: footprint (none) -> Diode_SMD:D_SOD-323_HandSoldering
- J101: footprint (none) -> Connector_Coaxial:SMA_Amphenol_132134_Vertical
Connections:
- net GND_ISO is gone; now on net GND: U1.1 (GND), U1.11 (GND), U1.12 (GND)
- net 3V3: now also R109.1
- net GPS_ENABLE: now also U1.24 (P1.07)
- net GPS_RX: now also U1.30 (P1.06), U103.1 (B2); no longer U103.8 (B1)
- net GPS_TX: now also U1.31 (P0.27), U103.8 (B1); no longer U103.1 (B2)
- net MCP_INT: now also U1.3 (P1.03)
- net MCP_RST: now also U1.22 (P0.20)
- net MCP_SPI_CS: now also U1.55 (P1.04), R109.2
- net MCP_SPI_MISO: now also R106.2
- net MCP_SPI_MOSI: now also R107.2
- net MCP_SPI_SCK: now also R108.2
- net ublox/GPS_RX: now also U103.4 (A2); no longer U103.5 (A1)
- net ublox/GPS_TX: now also U103.5 (A1); no longer U103.4 (A2)
- net at U1.10 (P1.02): now also R108.1
- net RST: now reaches U1.32 (RST)
- net at U1.8 (P1.00): now also R106.1
- net at U1.9 (P1.01): now also R107.1

Commit message: redesing board
Parts:
- added C110, C112: 10nF, Capacitor_SMD:C_0603_1608Metric, symbol Device:C_Small
- added C111: 10uF, Capacitor_SMD:C_0603_1608Metric, symbol Device:C_Small
- added C114: 2.2uF, Capacitor_SMD:C_0603_1608Metric, symbol Device:C_Small
- added D102, D103: WS2812B-2020, LED_SMD:LED_WS2812B-2020_PLCC4_2.0x2.0mm, symbol LED:WS2812B-2020
- added D104: BZT52C16S, Diode_SMD:D_SOD-323_HandSoldering, symbol Device:D_Zener_Small
- added H101, H102: MountingHole_Pad, MountingHole:MountingHole_2.2mm_M2_Pad_Via, symbol Mechanical:MountingHole_Pad
- added J102: Vin, Connector_PinHeader_2.54mm:PinHeader_1x01_P2.54mm_Vertical, symbol Connector_Generic:Conn_01x01
- added J103: Gnd, Connector_PinHeader_2.54mm:PinHeader_1x01_P2.54mm_Vertical, symbol Connector_Generic:Conn_01x01
- added Q101: AO3401A, Package_TO_SOT_SMD:SOT-23, symbol Transistor_FET:AO3401A
- added R107: 10K, Resistor_SMD:R_0603_1608Metric, symbol Device:R_Small
- added TP101: 5V, TestPoint:TestPoint_Pad_1.0x1.0mm, symbol Connector:TestPoint
- added TP102: 3V3, TestPoint:TestPoint_Pad_1.0x1.0mm, symbol Connector:TestPoint
- added U105: LP2985-3.3, Package_TO_SOT_SMD:SOT-23-5, symbol Regulator_Linear:LP2985-3.3
- C104: footprint Capacitor_THT:CP_Radial_D5.0mm_P2.50mm -> Capacitor_THT:CP_Radial_D8.0mm_P3.50mm
- renumbered C6 to C101, C3 to C102, C5 to C103, C4 to C105, C102 to C107, C105 to C108, C101 to C109, C1 to C113, C2 to C115, J3 to J104, JP102 to JP101, R109 to R101, R104 to R102, R105 to R103, R101 to R104, R102 to R105, R103 to R106, R106 to R108, R108 to R109, R107 to R110, U2 to U101, U103 to U102, U102 to U103, U1 to U104, Y1 to Y101
Connections:
- net 3V3: now also C114.1, TP102.1, U105.5 (VOUT)
- net 5V: now also C111.1, D102.4 (VDD), D103.4 (VDD), TP101.1, U105.1 (VIN), U105.3 (ON/~{OFF})
- net CAN_TERM: now also U104.22 (P0.20)
- net GND: now also J104.6 (Pin_6), J104.9 (Pin_9), C110.2, C111.2, C112.2, C114.2, D102.2 (VSS), D103.2 (VSS), H101.1, H102.1, J103.1 (Pin_1), R107.2, U105.2 (GND)
- net GPS_ENABLE: now also U104.19 (P0.15_(QSPI)); no longer U104.24 (P1.07)
- net GPS_RX: now also U104.9 (P1.01); no longer U104.30 (P1.06)
- net GPS_TX: now also U104.10 (P1.02); no longer U104.31 (P0.27)
- net MCP_INT: now also U104.24 (P1.07); no longer U104.3 (P1.03)
- net MCP_RST: now also U104.25 (P1.09); no longer U104.22 (P0.20)
- net MCP_SPI_CS: now also U104.28 (P0.19); no longer U104.55 (P1.04)
- net RST: now also J104.2 (Pin_2)
- net at R109.1: now also U104.31 (P0.27); no longer U104.10 (P1.02)
- net at U104.29 (P0.21): now also R108.1
- net LED_CONTROL: now reaches U104.8 (P1.00)
- net LED_CONTROL: now also D102.3 (DIN); no longer R108.1
- net at R110.1: now also U104.30 (P1.06); no longer U104.9 (P1.01)
- new net: C112.1, U105.4 (BP)
- new net: D102.1 (DOUT), D103.3 (DIN)
- new net: C110.1, D104.2 (A), Q101.1 (G), R107.1
- new net 12V: D104.1 (K), Q101.2 (S)
- new net VIN: J102.1 (Pin_1), Q101.3 (D)
Other:
- added sheet lmr16006 (lmr16006.kicad_sch)
- note added: "MCU"
- note added: "POWER"
- moved on the sheet: C101, C102, C103, C105, C113, C115, J104, JP101, R101, R103, R104, R108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

Commit message: wip
Connections:
- net GPS_RX: now also U102.8 (B1), U104.10 (P1.02); no longer U102.1 (B2), U104.9 (P1.01)
- net GPS_TX: now also U102.1 (B2), U104.9 (P1.01); no longer U102.8 (B1), U104.10 (P1.02)
- net ublox/GPS_RX: now also U102.5 (A1); no longer U102.4 (A2)
- net ublox/GPS_TX: now also U102.4 (A2); no longer U102.5 (A1)
Changed lines of the file:
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@@
 	(wire
 		(pts
-			(xy 50.8 162.56) (xy 50.8 139.7)
-		)
-		(stroke
-			(width 0)
-			(type default)
-		)
-	)
-	(wire
-		(pts
 			(xy 151.13 85.09) (xy 147.32 85.09)
 		)
@@
 	(wire
 		(pts
+			(xy 49.53 158.75) (xy 49.53 134.62)
+		)
+		(stroke
+			(width 0)
+			(type default)
+		)
+	)
+	(wire
+		(pts
 			(xy 54.61 115.57) (xy 54.61 116.84)
 		)
@@
 	(wire
 		(pts
-			(xy 50.8 139.7) (xy 66.04 139.7)
-		)
-		(stroke
-			(width 0)
-			(type default)
-		)
-	)
-	(wire
-		(pts
 			(xy 261.62 16.51) (xy 271.78 16.51)
 		)
@@
 	(wire
 		(pts
-			(xy 46.99 157.48) (xy 46.99 134.62)
-		)
-		(stroke
-			(width 0)
-			(type default)
-		)
-	)
-	(wire
-		(pts
 			(xy 59.69 176.53) (xy 72.39 176.53)
 		)
@@
 	(wire
 		(pts
-			(xy 35.56 157.48) (xy 46.99 157.48)
+			(xy 147.32 31.75) (xy 158.75 31.75)
 		)
 		(stroke
@@
 	(wire
 		(pts
-			(xy 147.32 31.75) (xy 158.75 31.75)
+			(xy 77.47 53.34) (xy 102.87 53.34)
 		)
 		(stroke
@@
 	(wire
 		(pts
-			(xy 77.47 53.34) (xy 102.87 53.34)
+			(xy 259.08 90.17) (xy 281.94 90.17)
 		)
 		(stroke
@@
 	(wire
 		(pts
-			(xy 259.08 90.17) (xy 281.94 90.17)
+			(xy 55.88 139.7) (xy 66.04 139.7)
 		)
 		(stroke
@@
 	(wire
 		(pts
-			(xy 46.99 134.62) (xy 66.04 134.62)
-		)
-		(stroke
-			(width 0)
-			(type default)
-		)
-	)
-	(wire
-		(pts
 			(xy 147.32 24.13) (xy 158.75 24.13)
 		)
@@
 	(wire
 		(pts
+			(xy 49.53 134.62) (xy 66.04 134.62)
+		)
+		(stroke
+			(width 0)
+			(type default)
+		)
+	)
+	(wire
+		(pts
 			(xy 226.06 147.32) (xy 228.6 147.32)
 		)
@@
 	(wire
 		(pts
+			(xy 35.56 161.29) (xy 55.88 161.29)
+		)
+		(stroke
+			(width 0)
+			(type default)
+		)
+	)
+	(wire
+		(pts
 			(xy 22.86 58.42) (xy 46.99 58.42)
 		)
@@
 	(wire
 		(pts
+			(xy 35.56 158.75) (xy 49.53 158.75)
+		)
+		(stroke
+			(width 0)
+			(type default)
+		)
+	)
+	(wire
+		(pts
 			(xy 259.08 97.79) (xy 281.94 97.79)
 		)
@@
 	(wire
 		(pts
+			(xy 55.88 161.29) (xy 55.88 139.7)
+		)
+		(stroke
+			(width 0)
+			(type default)
+		)
+	)
+	(wire
+		(pts
 			(xy 168.91 147.32) (xy 183.642 147.32)
 		)
@@
 	(wire
 		(pts
-			(xy 35.56 162.56) (xy 50.8 162.56)
-		)
-		(stroke
-			(width 0)
-			(type default)
-		)
-	)
-	(wire
-		(pts
 			(xy 41.91 82.55) (xy 41.91 85.09)
 		)
@@
 	)
 	(label "GPS_TX"
-		(at 281.94 40.64 180)
+		(at 281.94 38.1 180)
 		(effects
 			(font
@@
 	)
 	(label "GPS_RX"
-		(at 97.79 139.7 180)
+		(at 97.79 134.62 180)
 		(effects
 			(font
@@
 	)
 	(label "GPS_RX"
-		(at 281.94 38.1 180)
+		(at 281.94 40.64 180)
 		(effects
 			(font
@@
 	)
 	(label "GPS_TX"
-		(at 97.79 134.62 180)
+		(at 97.79 139.7 180)
 		(effects
 			(font
@@
 		)
 		(pin "GPS_RX" input
-			(at 35.56 162.56 0)
+			(at 35.56 158.75 0)
 			(effects
 				(font
@@
 		)
 		(pin "GPS_TX" input
-			(at 35.56 157.48 0)
+			(at 35.56 161.29 0)
 			(effects
 				(font

Commit message: wip
Parts:
- added LOGO101: ~, logo:logo_github, symbol logo:logo_qr_github
- added LOGO102: ~, logo:logo_15x9, symbol logo:logo15x9
Other:
- moved on the sheet: H101, H102
Changed lines of the file:
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@@
 	(wire
 		(pts
-			(xy 154.94 111.76) (xy 154.94 115.57)
+			(xy 154.94 118.11) (xy 154.94 121.92)
 		)
 		(stroke
@@
 	(wire
 		(pts
-			(xy 144.78 111.76) (xy 144.78 115.57)
+			(xy 144.78 118.11) (xy 144.78 121.92)
 		)
 		(stroke
@@
 	(symbol
 		(lib_id "power:GND")
-		(at 144.78 115.57 0)
+		(at 144.78 121.92 0)
 		(unit 1)
 		(exclude_from_sim no)
@@
 		(dnp no)
 		(property "Reference" "#PWR0118"
-			(at 144.78 121.92 0)
+			(at 144.78 128.27 0)
 			(effects
 				(font
@@
 		)
 		(property "Value" "GND"
-			(at 144.907 119.9642 0)
+			(at 144.907 126.3142 0)
 			(effects
 				(font
@@
 		)
 		(property "Footprint" ""
-			(at 144.78 115.57 0)
+			(at 144.78 121.92 0)
 			(effects
 				(font
@@
 		)
 		(property "Datasheet" ""
-			(at 144.78 115.57 0)
+			(at 144.78 121.92 0)
 			(effects
 				(font
@@
 		)
 		(property "Description" ""
-			(at 144.78 115.57 0)
+			(at 144.78 121.92 0)
 			(effects
 				(font
@@
 	(symbol
 		(lib_id "Mechanical:MountingHole_Pad")
-		(at 154.94 109.22 0)
+		(at 154.94 115.57 0)
 		(unit 1)
 		(exclude_from_sim no)
@@
 		(dnp no)
 		(property "Reference" "H102"
-			(at 157.988 106.68 0)
+			(at 153.162 110.744 0)
 			(effects
 				(font
@@
 		)
 		(property "Value" "MountingHole_Pad"
-			(at 157.48 109.2199 0)
+			(at 151.638 126.746 90)
 			(effects
 				(font
@@
 		)
 		(property "Footprint" "MountingHole:MountingHole_2.2mm_M2_Pad_Via"
-			(at 154.94 109.22 0)
+			(at 154.94 115.57 0)
 			(effects
 				(font
@@
 		)
 		(property "Datasheet" "~"
-			(at 154.94 109.22 0)
+			(at 154.94 115.57 0)
 			(effects
 				(font
@@
 		)
 		(property "Description" "Mounting Hole with connection"
-			(at 154.94 109.22 0)
+			(at 154.94 115.57 0)
 			(effects
 				(font
@@
 	)
 	(symbol
+		(lib_id "logo:logo15x9")
+		(at 173.99 127 0)
+		(unit 1)
+		(exclude_from_sim no)
+		(in_bom no)
+		(on_board yes)
+		(dnp no)
+		(property "Reference" "LOGO102"
+			(at 174.752 116.84 0)
+			(effects
+				(font
+					(size 1.27 1.27)
+				)
+				(justify left)
+			)
+		)
+		(property "Value" "~"
+			(at 184.15 124.4599 0)
+			(effects
+				(font
+					(size 1.27 1.27)
+				)
+				(justify left)
+			)
+		)
+		(property "Footprint" "logo:logo_15x9"
+			(at 173.99 127 0)
+			(effects
+				(font
+					(size 1.27 1.27)
+				)
+				(hide yes)
+			)
+		)
+		(property "Datasheet" ""
+			(at 173.99 127 0)
+			(effects
+				(font
+					(size 1.27 1.27)
+				)
+				(hide yes)
+			)
+		)
+		(property "Description" ""
+			(at 173.99 127 0)
+			(effects
+				(font
+					(size 1.27 1.27)
+				)
+				(hide yes)
+			)
+		)
+		(instances
+			(project ""
+				(path "/48fe87cd-0661-436a-93bb-f175c4d0f54e"
+					(reference "LOGO102")
+					(unit 1)
+				)
+			)
+		)
+	)
+	(symbol
 		(lib_id "Device:R_Small")
 		(at 204.47 83.82 270)
@@
 	)
 	(symbol
+		(lib_id "logo:logo_qr_github")
+		(at 166.37 123.19 0)
+		(unit 1)
+		(exclude_from_sim no)
+		(in_bom yes)
+		(on_board yes)
+		(dnp no)
+		(property "Reference" "LOGO101"
+			(at 162.56 114.3 0)
+			(effects
+				(font
+					(size 1.27 1.27)
+				)
+				(justify left)
+			)
+		)
+		(property "Value" "~"
+			(at 172.72 122.5125 0)
+			(effects
+				(font
+					(size 1.27 1.27)
+				)
+				(justify left)
+			)
+		)
+		(property "Footprint" "logo:logo_github"
+			(at 166.624 130.302 0)
+			(effects
+				(font
+					(size 1.27 1.27)
+				)
+				(hide yes)
+			)
+		)
+		(property "Datasheet" ""
+			(at 166.37 123.19 0)
+			(effects
+				(font
+					(size 1.27 1.27)
+				)
+				(hide yes)
+			)
+		)
+		(property "Description" ""
+			(at 166.37 123.19 0)
+			(effects
+				(font
+					(size 1.27 1.27)
+				)
+				(hide yes)
+			)
+		)
+		(instances
+			(project ""
+				(path "/48fe87cd-0661-436a-93bb-f175c4d0f54e"
+					(reference "LOGO101")
+					(unit 1)
+				)
+			)
+		)
+	)
+	(symbol
 		(lib_id "power:GND")
 		(at 76.2 154.94 0)
@@
 	(symbol
 		(lib_id "Mechanical:MountingHole_Pad")
-		(at 144.78 109.22 0)
+		(at 144.78 115.57 0)
 		(unit 1)
 		(exclude_from_sim no)
@@
 		(dnp no)
 		(property "Reference" "H101"
-			(at 143.256 100.838 0)
+			(at 142.494 110.744 0)
 			(effects
 				(font
@@
 		)
 		(property "Value" "MountingHole_Pad"
-			(at 139.192 103.886 0)
+			(at 140.716 127 90)
 			(effects
 				(font
@@
 		)
 		(property "Footprint" "MountingHole:MountingHole_2.2mm_M2_Pad_Via"
-			(at 144.78 109.22 0)
+			(at 144.78 115.57 0)
 			(effects
 				(font
@@
 		)
 		(property "Datasheet" "~"
-			(at 144.78 109.22 0)
+			(at 144.78 115.57 0)
 			(effects
 				(font
@@
 		)
 		(property "Description" "Mounting Hole with connection"
-			(at 144.78 109.22 0)
+			(at 144.78 115.57 0)
 			(effects
 				(font
@@
 	(symbol
 		(lib_id "power:GND")
-		(at 154.94 115.57 0)
+		(at 154.94 121.92 0)
 		(unit 1)
 		(exclude_from_sim no)
@@
 		(dnp no)
 		(property "Reference" "#PWR0121"
-			(at 154.94 121.92 0)
+			(at 154.94 128.27 0)
 			(effects
 				(font
@@
 		)
 		(property "Value" "GND"
-			(at 155.067 119.9642 0)
+			(at 155.067 126.3142 0)
 			(effects
 				(font
@@
 		)
 		(property "Footprint" ""
-			(at 154.94 115.57 0)
+			(at 154.94 121.92 0)
 			(effects
 				(font
@@
 		)
 		(property "Datasheet" ""
-			(at 154.94 115.57 0)
+			(at 154.94 121.92 0)
 			(effects
 				(font
@@
 		)
 		(property "Description" ""
-			(at 154.94 115.57 0)
+			(at 154.94 121.92 0)
 			(effects
 				(font

Commit message: VDDH pin
Connections:
- net 3V3: now also U104.14 (VDDH)
- no-connect marks 5 -> 7
Changed lines of the file:
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@@
+	)
+	(junction
+		(at 245.11 16.51)
+		(diameter 0)
+		(color 0 0 0 0)
 	)
 	(junction
@@
 		(diameter 0)
 		(color 0 0 0 0)
+	)
+	(no_connect
+		(at 231.14 24.13)
 	)
 	(no_connect
@@
 	)
 	(no_connect
+		(at 226.06 24.13)
+	)
+	(no_connect
 		(at 77.47 55.88)
 	)
@@
 	(wire
 		(pts
+			(xy 238.76 24.13) (xy 238.76 16.51)
+		)
+		(stroke
+			(width 0)
+			(type default)
+		)
+	)
+	(wire
+		(pts
 			(xy 43.18 115.57) (xy 54.61 115.57)
 		)
@@
 		)
 		(stroke
+			(width 0)
+			(type default)
+		)
+	)
+	(wire
+		(pts
+			(xy 238.76 16.51) (xy 245.11 16.51)
+		)
+		(stroke

Commit message: PCBA ready
Parts:
- C101, C103: value 12pF -> 8pF
Changed lines of the file:
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@@
 			)
 		)
-		(property "Value" "12pF"
+		(property "Value" "8pF"
 			(at 45.339 83.5723 0)
 			(effects
@@
 			)
 		)
-		(property "Value" "12pF"
+		(property "Value" "8pF"
 			(at 21.082 84.074 0)
 			(effects
