File: ubloxM8N.kicad_sch (KiCad schematic)
At the start: 5 parts, among them U17 NEO-8M

Commit message: redesing board
Parts:
- L201: renamed from L2; footprint Inductor_SMD:L_0805_2012Metric_Pad1.15x1.40mm_HandSolder -> Inductor_SMD:L_0805_2012Metric
- R201: renamed from R40; footprint Resistor_SMD:R_1206_3216Metric -> Resistor_SMD:R_0603_1608Metric
- renumbered C40 to C201, C49 to C202, U17 to U201
Changed lines of the file:
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@@
 		(on_board yes)
 		(dnp no)
-		(property "Reference" "U17"
+		(property "Reference" "U201"
 			(at 143.51 64.3382 0)
 			(effects
@@
 			(project "dash"
 				(path "/48fe87cd-0661-436a-93bb-f175c4d0f54e/5b68915a-9fa4-45be-9b08-ed6751f5983f"
-					(reference "U17")
+					(reference "U201")
 					(unit 1)
 				)
@@
 		(on_board yes)
 		(dnp no)
-		(property "Reference" "L2"
+		(property "Reference" "L201"
 			(at 106.7562 77.5716 0)
 			(effects
@@
 			)
 		)
-		(property "Footprint" "Inductor_SMD:L_0805_2012Metric_Pad1.15x1.40mm_HandSolder"
+		(property "Footprint" "Inductor_SMD:L_0805_2012Metric"
 			(at 105.41 78.74 0)
 			(effects
@@
 			(project "dash"
 				(path "/48fe87cd-0661-436a-93bb-f175c4d0f54e/5b68915a-9fa4-45be-9b08-ed6751f5983f"
-					(reference "L2")
+					(reference "L201")
 					(unit 1)
 				)
@@
 		(on_board yes)
 		(dnp no)
-		(property "Reference" "C40"
+		(property "Reference" "C201"
 			(at 107.7468 89.0016 0)
 			(effects
@@
 			(project "dash"
 				(path "/48fe87cd-0661-436a-93bb-f175c4d0f54e/5b68915a-9fa4-45be-9b08-ed6751f5983f"
-					(reference "C40")
+					(reference "C201")
 					(unit 1)
 				)
@@
 		(on_board yes)
 		(dnp no)
-		(property "Reference" "R40"
+		(property "Reference" "R201"
 			(at 97.79 79.8322 90)
 			(effects
@@
 			)
 		)
-		(property "Footprint" "Resistor_SMD:R_1206_3216Metric"
+		(property "Footprint" "Resistor_SMD:R_0603_1608Metric"
 			(at 97.79 83.312 90)
 			(effects
@@
 			(project "dash"
 				(path "/48fe87cd-0661-436a-93bb-f175c4d0f54e/5b68915a-9fa4-45be-9b08-ed6751f5983f"
-					(reference "R40")
+					(reference "R201")
 					(unit 1)
 				)
@@
 		(on_board yes)
 		(dnp no)
-		(property "Reference" "C49"
+		(property "Reference" "C202"
 			(at 176.3268 72.4916 0)
 			(effects
@@
 			(project "dash"
 				(path "/48fe87cd-0661-436a-93bb-f175c4d0f54e/5b68915a-9fa4-45be-9b08-ed6751f5983f"
-					(reference "C49")
-					(unit 1)
-				)
+					(reference "C202")
+					(unit 1)
+				)

Commit message: PCBA ready
Parts:
- C201: value 0.01uF -> 10nF
Changed lines of the file:
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@@
 			)
 		)
-		(property "Value" "0.01uF"
+		(property "Value" "10nF"
 			(at 107.7468 91.313 0)
 			(effects
